Commit message: using limited joint config. still need ee fixed

File: urdf/custom_ur5.urdf.xacro (robot description, xacro)
@@ -8,5 +8,14 @@
   <xacro:include filename="$(find ur_description)/urdf/ur5.urdf.xacro" />
   <!-- arm -->
-  <xacro:ur5_robot prefix="" joint_limited="false"
+  <!-- <xacro:ur5_robot prefix="" joint_limited="false"
+    transmission_hw_interface="$(arg transmission_hw_interface)"
+  /> -->
+  <xacro:ur5_robot prefix="" joint_limited="true"
+    shoulder_pan_lower_limit="${-pi}" shoulder_pan_upper_limit="${pi}"
+    shoulder_lift_lower_limit="${-pi}" shoulder_lift_upper_limit="${pi}"
+    elbow_joint_lower_limit="${-pi}" elbow_joint_upper_limit="${pi}"
+    wrist_1_lower_limit="${-pi}" wrist_1_upper_limit="${pi}"
+    wrist_2_lower_limit="${-pi}" wrist_2_upper_limit="${pi}"
+    wrist_3_lower_limit="${-pi}" wrist_3_upper_limit="${pi}"
     transmission_hw_interface="$(arg transmission_hw_interface)"
   />
@@ -54,7 +63,7 @@
     <parent link="dummy_link" />
     <child link = "base_link" />
-    <origin xyz="0.0 0.0 1.21207" rpy="0.0 0.0 0.0" />
+    <origin xyz="0.0 0.0 1.01207" rpy="0.0 0.0 0.0" />
   </joint>
- <joint name="robotiq_joint" type="fixed">
+ <!-- <joint name="robotiq_joint" type="fixed">
     <parent link="ee_link" />
     <child link = "robotiq_arg2f_base_link" />
@@ -63,4 +72,4 @@
 <xacro:include filename="$(find robotiq_2f_85_gripper_visualization)/urdf/robotiq_arg2f_transmission.xacro" />
 <xacro:include filename="$(find robotiq_2f_85_gripper_visualization)/urdf/robotiq_arg2f_85_model_macro.xacro" />
-<xacro:robotiq_arg2f_85 prefix=""/>
+<xacro:robotiq_arg2f_85 prefix=""/> -->
 </robot>

Commit message: working joint limits

File: urdf/custom_ur5.urdf.xacro (robot description, xacro)
@@ -13,5 +13,5 @@
   <xacro:ur5_robot prefix="" joint_limited="true"
     shoulder_pan_lower_limit="${-pi}" shoulder_pan_upper_limit="${pi}"
-    shoulder_lift_lower_limit="${-pi}" shoulder_lift_upper_limit="${pi}"
+    shoulder_lift_lower_limit="${-pi}" shoulder_lift_upper_limit="${-pi/4}"
     elbow_joint_lower_limit="${-pi}" elbow_joint_upper_limit="${pi}"
     wrist_1_lower_limit="${-pi}" wrist_1_upper_limit="${pi}"

File: urdf/kdl_custom_ur5.urdf (robot description, URDF)
Before this commit: robot ur5, 12 links, 11 joints
Joints:
- joint shoulder_lift_joint: limit lower=-3.14159265359 upper=3.14159265359 effort=150.0 velocity=3.15 -> lower=-3.14159265359 upper=-0.785398163397 effort=150.0 velocity=3.15

Commit message: bare bone gripper working

File: urdf/custom_ur5.urdf.xacro (robot description, xacro)
@@ -65,11 +65,44 @@
     <origin xyz="0.0 0.0 1.01207" rpy="0.0 0.0 0.0" />
   </joint>
- <!-- <joint name="robotiq_joint" type="fixed">
-    <parent link="ee_link" />
+  <!-- <xacro:include filename="$(find ur5_intpro)/urdf/robotiq_arg2f_transmission.xacro" />
+  <xacro:include filename="$(find ur5_intpro)/urdf/robotiq_arg2f_85_model_macro.xacro" />
+  <xacro:robotiq_arg2f_85 prefix=""/>
+  <xacro:robotiq_arg2f_transmission prefix="" />
+  <joint name="robotiq_joint" type="fixed">
+    <parent link="tool0" />
     <child link = "robotiq_arg2f_base_link" />
-    <origin xyz="0 0 0" rpy="0.0 0.0 0.0" />
- </joint>
-<xacro:include filename="$(find robotiq_2f_85_gripper_visualization)/urdf/robotiq_arg2f_transmission.xacro" />
-<xacro:include filename="$(find robotiq_2f_85_gripper_visualization)/urdf/robotiq_arg2f_85_model_macro.xacro" />
-<xacro:robotiq_arg2f_85 prefix=""/> -->
+    <origin xyz="0.0 0.0 0.0" rpy="0.0 0.0 0.0" />
+ </joint> -->
+<!--  <link name="robotiq_arg2f_base_link">
+    <inertial>
+      <origin xyz="0 0 0" rpy="0 0 0" />
+      <mass value="0.48" />
+      <inertia
+        ixx="6.66"
+        ixy="0"
+        ixz="0"
+        iyy="6.66"
+        iyz="0"
+        izz="6.66" />
+    </inertial>
+     <visual>
+      <geometry>
+        <box size="0.05 0.05 0.05"/>
+      </geometry>
+      <origin rpy="0 0 0" xyz="0 0 0"/>
+    </visual>
+    <collision>
+      <geometry>
+        <box size="0.05 0.05 0.05"/>
+      </geometry>
+      <origin rpy="0 0 0" xyz="0 0 0"/>
+    </collision>
+  </link>
+   <gazebo reference="robotiq_arg2f_base_link">
+    <mu1 value="1.0"/>
+    <mu2 value="1.0"/>
+    <kp value="900000000.0"></kp>
+    <kd value="800000000.0"></kd>
+    <selfCollide value="false"/>
+  </gazebo> -->
 </robot>

Commit message: adding original urdf to this package

File: urdf/custom_ur5.urdf.xacro (robot description, xacro)
@@ -4,7 +4,7 @@
   <xacro:arg name="transmission_hw_interface" default="hardware_interface/PositionJointInterface"/>
   <!-- common stuff -->
-  <xacro:include filename="$(find ur_description)/urdf/common.gazebo.xacro" />
+  <xacro:include filename="$(find ur5_intpro)/urdf/common.gazebo.xacro" />
   <!-- ur5 -->
-  <xacro:include filename="$(find ur_description)/urdf/ur5.urdf.xacro" />
+  <xacro:include filename="$(find ur5_intpro)/urdf/ur5.urdf.xacro" />
   <!-- arm -->
   <!-- <xacro:ur5_robot prefix="" joint_limited="false"
@@ -65,13 +65,53 @@
     <origin xyz="0.0 0.0 1.01207" rpy="0.0 0.0 0.0" />
   </joint>
-  <!-- <xacro:include filename="$(find ur5_intpro)/urdf/robotiq_arg2f_transmission.xacro" />
-  <xacro:include filename="$(find ur5_intpro)/urdf/robotiq_arg2f_85_model_macro.xacro" />
-  <xacro:robotiq_arg2f_85 prefix=""/>
-  <xacro:robotiq_arg2f_transmission prefix="" />
+  <!-- <xacro:include filename="$(find ur5_intpro)/urdf/robotiq_arg2f_transmission.xacro" /> -->
+  <!-- <xacro:include filename="$(find ur5_intpro)/urdf/robotiq_arg2f_85_model_macro.xacro" /> -->
+  <!-- <xacro:robotiq_arg2f_85 prefix=""/> -->
+  <!-- <xacro:robotiq_arg2f_transmission prefix="" /> -->
+  <link name="robotiq_arg2f_base_link">
+      <!-- <inertial>
+        <origin xyz="8.625E-08 -4.6583E-06 0.03145" rpy="0 0 0" />
+        <mass value="10.22652" />
+        <inertia ixx="0.020005" ixy="-4.2442E-10" ixz="-2.9069E-10" iyy="0.17832" iyz="-3.4402E-08" izz="0.013478" />
+      </inertial> -->
+      <inertial>
+      <origin xyz="0 0 0" rpy="0 0 0" />
+      <mass value="0.48" />
+      <inertia
+        ixx="6.66"
+        ixy="0"
+        ixz="0"
+        iyy="6.66"
+        iyz="0"
+        izz="6.66" />
+    </inertial>
+      <visual>
+        <origin xyz="0 0 0" rpy="0 0 0" />
+        <geometry>
+        <!-- <box size="0.05 0.05 0.05"/> -->
+          <!-- <mesh filename="package://ur5_intpro/meshes/visual/robotiq_arg2f_85_base_link_1.dae"/> -->
+          <mesh filename="package://ur5_intpro/meshes/visual/base.dae"/>
+        </geometry>
+      </visual>
+      <collision>
+        <origin xyz="0 0 0" rpy="0 0 0" />
+        <geometry>
+        <!-- <box size="0.05 0.05 0.05"/> -->
+           <!-- <mesh filename="package://ur5_intpro/meshes/visual/robotiq_arg2f_85_base_link_1.dae" /> -->
+           <mesh filename="package://ur5_intpro/meshes/visual/base.dae" />
+        </geometry>
+      </collision>
+    </link>
   <joint name="robotiq_joint" type="fixed">
     <parent link="tool0" />
     <child link = "robotiq_arg2f_base_link" />
-    <origin xyz="0.0 0.0 0.0" rpy="0.0 0.0 0.0" />
- </joint> -->
+    <origin xyz="0.5 0.0 0.5" rpy="0.0 0.0 0.0" />
+ </joint>
+<gazebo reference="robotiq_arg2f_base_link">
+      <mu1 value="1.0"/>
+      <mu2 value="1.0"/>
+      <kp value="900000000.0"></kp>
+      <kd value="800000000.0"></kd>
+  </gazebo>
 <!--  <link name="robotiq_arg2f_base_link">
     <inertial>

File: urdf/kdl_custom_ur5.urdf (robot description, URDF)
Before this commit: robot ur5, 12 links, 11 joints
Links:
- added link robotiq_arg2f_base_link, mass 0.48; collision mesh filename=package://ur5_intpro/meshes/visual/base.dae; visual mesh filename=package://ur5_intpro/meshes/visual/base.dae
Joints:
- added joint robotiq_joint: type fixed, parent tool0, child robotiq_arg2f_base_link, origin xyz=0.5 0.0 0.5 rpy=0.0 0.0 0.0

File: urdf/robotiq_arg2f.xacro (robot description, xacro)
@@ -5,29 +5,29 @@
       <inertial>
         <origin xyz="8.625E-08 -4.6583E-06 0.03145" rpy="0 0 0" />
-        <mass value="0.22652" />
-        <inertia ixx="0.00020005" ixy="-4.2442E-10" ixz="-2.9069E-10" iyy="0.00017832" iyz="-3.4402E-08" izz="0.00013478" />
+        <mass value="10.22652" />
+        <inertia ixx="0.020005" ixy="-4.2442E-10" ixz="-2.9069E-10" iyy="0.17832" iyz="-3.4402E-08" izz="0.013478" />
       </inertial>
       <visual>
         <origin xyz="0 0 0" rpy="0 0 0" />
         <geometry>
-          <mesh filename="package://ur5_intpro/meshes/visual/robotiq_arg2f_85_base_link.dae" scale="0.001 0.001 0.001"/>
+          <mesh filename="package://ur5_intpro/meshes/visual/robotiq_arg2f_85_base_link.dae"/>
         </geometry>
-        <material name="">
+        <!-- <material name="">
           <color rgba="0.1 0.1 0.1 1" />
-        </material>
+        </material> -->
       </visual>
       <collision>
         <origin xyz="0 0 0" rpy="0 0 0" />
         <geometry>
-           <mesh filename="package://ur5_intpro/meshes/collision/robotiq_arg2f_base_link.stl" />
+           <mesh filename="package://ur5_intpro/meshes/visual/robotiq_arg2f_85_base_link.dae" />
         </geometry>
       </collision>
     </link>
-    <gazebo reference="${prefix}robotiq_arg2f_base_link">
+    <!-- <gazebo reference="${prefix}robotiq_arg2f_base_link">
       <mu1 value="1.0"/>
       <mu2 value="1.0"/>
       <kp value="900000000.0"></kp>
       <kd value="800000000.0"></kd>
-    </gazebo>
+    </gazebo> -->
   </xacro:macro>
   <xacro:macro name="finger_joints" params="prefix fingerprefix reflect">

File: urdf/robotiq_arg2f_85_model_macro.xacro (robot description, xacro)
@@ -12,5 +12,5 @@
         <origin xyz="0 0 0" rpy="0 0 0" />
         <geometry>
-          <mesh filename="package://ur5_intpro/meshes/gripper/visual/robotiq_arg2f_85_outer_knuckle.dae" scale="0.001 0.001 0.001"/>
+          <mesh filename="package://ur5_intpro/meshes/gripper/visual/robotiq_arg2f_85_outer_knuckle.dae" scale="1 1 1"/>
         </geometry>
         <material name="">
@@ -21,5 +21,5 @@
         <origin xyz="0 0 0" rpy="0 0 0" />
         <geometry>
-          <mesh filename="package://ur5_intpro/meshes/gripper/collision/robotiq_arg2f_85_outer_knuckle.dae" scale="0.001 0.001 0.001"/>
+          <mesh filename="package://ur5_intpro/meshes/gripper/visual/robotiq_arg2f_85_outer_knuckle.dae" scale="1 1 1"/>
         </geometry>
       </collision>
@@ -42,5 +42,5 @@
         <origin xyz="0 0 0" rpy="0 0 0" />
         <geometry>
-          <mesh filename="package://ur5_intpro/meshes/gripper/visual/robotiq_arg2f_85_outer_finger.dae" scale="0.001 0.001 0.001"/>
+          <mesh filename="package://ur5_intpro/meshes/gripper/visual/robotiq_arg2f_85_outer_finger.dae" scale="1 1 1"/>
         </geometry>
         <material name="">
@@ -51,5 +51,5 @@
         <origin xyz="0 0 0" rpy="0 0 0" />
         <geometry>
-          <mesh filename="package://ur5_intpro/meshes/gripper/collision/robotiq_arg2f_85_outer_finger.dae" scale="0.001 0.001 0.001"/>
+          <mesh filename="package://ur5_intpro/meshes/gripper/visual/robotiq_arg2f_85_outer_finger.dae" scale="1 1 1"/>
         </geometry>
       </collision>
@@ -72,5 +72,5 @@
         <origin xyz="0 0 0" rpy="0 0 0" />
         <geometry>
-          <mesh filename="package://ur5_intpro/meshes/gripper/visual/robotiq_arg2f_85_inner_knuckle.dae" scale="0.001 0.001 0.001"/>
+          <mesh filename="package://ur5_intpro/meshes/gripper/visual/robotiq_arg2f_85_inner_knuckle.dae" scale="1 1 1"/>
         </geometry>
         <material name="">
@@ -81,5 +81,5 @@
         <origin xyz="0 0 0" rpy="0 0 0" />
         <geometry>
-          <mesh filename="package://ur5_intpro/meshes/gripper/collision/robotiq_arg2f_85_inner_knuckle.dae" scale="0.001 0.001 0.001"/>
+          <mesh filename="package://ur5_intpro/meshes/gripper/visual/robotiq_arg2f_85_inner_knuckle.dae" scale="1 1 1"/>
         </geometry>
       </collision>
@@ -102,5 +102,5 @@
         <origin xyz="0 0 0" rpy="0 0 0" />
         <geometry>
-          <mesh filename="package://ur5_intpro/meshes/gripper/visual/robotiq_arg2f_85_inner_finger.dae" scale="0.001 0.001 0.001"/>
+          <mesh filename="package://ur5_intpro/meshes/gripper/visual/robotiq_arg2f_85_inner_finger.dae" scale="1 1 1"/>
         </geometry>
         <material name="">
@@ -111,5 +111,5 @@
         <origin xyz="0 0 0" rpy="0 0 0" />
         <geometry>
-          <mesh filename="package://ur5_intpro/meshes/gripper/collision/robotiq_arg2f_85_inner_finger.dae" scale="0.001 0.001 0.001" />
+          <mesh filename="package://ur5_intpro/meshes/gripper/visual/robotiq_arg2f_85_inner_finger.dae" scale="1 1 1" />
         </geometry>
       </collision>

Commit message: fixed joint limit issue

File: urdf/custom_ur5.urdf.xacro (robot description, xacro)
@@ -13,6 +13,6 @@
   <xacro:ur5_robot prefix="" joint_limited="true"
     shoulder_pan_lower_limit="${-pi}" shoulder_pan_upper_limit="${pi}"
-    shoulder_lift_lower_limit="${-pi}" shoulder_lift_upper_limit="${-pi/4}"
-    elbow_joint_lower_limit="${-pi}" elbow_joint_upper_limit="${pi}"
+    shoulder_lift_lower_limit="${-pi/2.0}" shoulder_lift_upper_limit="${-pi/5.0}"
+    elbow_joint_lower_limit="${pi/5.0}" elbow_joint_upper_limit="${pi}"
     wrist_1_lower_limit="${-pi}" wrist_1_upper_limit="${pi}"
     wrist_2_lower_limit="${-pi}" wrist_2_upper_limit="${pi}"
@@ -20,4 +20,7 @@
     transmission_hw_interface="$(arg transmission_hw_interface)"
   />
+  <!-- shoulder_pan_lower_limit:=${-pi/3}    shoulder_pan_upper_limit:=${pi/3}
+    shoulder_lift_lower_limit:=${-pi/2.0}    shoulder_lift_upper_limit:=${-pi/2.0 + 0.01}
+    elbow_joint_lower_limit:=${-pi/3.0}    elbow_joint_upper_limit:=${0} -->
   <link name="world" />
   <joint name="dummy_joint" type="fixed">

File: urdf/kdl_custom_ur5.urdf (robot description, URDF)
Before this commit: robot ur5, 13 links, 12 joints
Joints:
- joint elbow_joint: limit lower=-3.14159265359 upper=3.14159265359 effort=150.0 velocity=3.15 -> lower=0.628318530718 upper=3.14159265359 effort=150.0 velocity=3.15
- joint shoulder_lift_joint: limit lower=-3.14159265359 upper=-0.785398163397 effort=150.0 velocity=3.15 -> lower=-1.57079632679 upper=-0.628318530718 effort=150.0 velocity=3.15

File: urdf/ur5.urdf.xacro (robot description, xacro)
@@ -13,7 +13,7 @@
   </xacro:macro>
   <xacro:macro name="ur5_robot" params="prefix joint_limited
-    shoulder_pan_lower_limit:=${-pi/3}    shoulder_pan_upper_limit:=${pi/3}
-    shoulder_lift_lower_limit:=${-pi/2.0}    shoulder_lift_upper_limit:=${-pi/2.0 + 0.01}
-    elbow_joint_lower_limit:=${-pi/3.0}    elbow_joint_upper_limit:=${0}
+    shoulder_pan_lower_limit:=${-pi}    shoulder_pan_upper_limit:=${pi}
+    shoulder_lift_lower_limit:=${-pi}    shoulder_lift_upper_limit:=${pi}
+    elbow_joint_lower_limit:=${-pi}    elbow_joint_upper_limit:=${pi}
     wrist_1_lower_limit:=${-pi}    wrist_1_upper_limit:=${pi}
     wrist_2_lower_limit:=${-pi}    wrist_2_upper_limit:=${pi}

Commit message: changed joint name

File: urdf/custom_ur5.urdf.xacro (robot description, xacro)
@@ -68,84 +68,73 @@
     <origin xyz="0.0 0.0 1.01207" rpy="0.0 0.0 0.0" />
   </joint>
-  <!-- <xacro:include filename="$(find ur5_intpro)/urdf/robotiq_arg2f_transmission.xacro" /> -->
-  <!-- <xacro:include filename="$(find ur5_intpro)/urdf/robotiq_arg2f_85_model_macro.xacro" /> -->
-  <!-- <xacro:robotiq_arg2f_85 prefix=""/> -->
-  <!-- <xacro:robotiq_arg2f_transmission prefix="" /> -->
-  <link name="robotiq_arg2f_base_link">
-      <!-- <inertial>
-        <origin xyz="8.625E-08 -4.6583E-06 0.03145" rpy="0 0 0" />
-        <mass value="10.22652" />
-        <inertia ixx="0.020005" ixy="-4.2442E-10" ixz="-2.9069E-10" iyy="0.17832" iyz="-3.4402E-08" izz="0.013478" />
-      </inertial> -->
-      <inertial>
-      <origin xyz="0 0 0" rpy="0 0 0" />
-      <mass value="0.48" />
-      <inertia
-        ixx="6.66"
-        ixy="0"
-        ixz="0"
-        iyy="6.66"
-        iyz="0"
-        izz="6.66" />
-    </inertial>
-      <visual>
-        <origin xyz="0 0 0" rpy="0 0 0" />
-        <geometry>
-        <!-- <box size="0.05 0.05 0.05"/> -->
-          <!-- <mesh filename="package://ur5_intpro/meshes/visual/robotiq_arg2f_85_base_link_1.dae"/> -->
-          <mesh filename="package://ur5_intpro/meshes/visual/base.dae"/>
-        </geometry>
-      </visual>
-      <collision>
-        <origin xyz="0 0 0" rpy="0 0 0" />
-        <geometry>
-        <!-- <box size="0.05 0.05 0.05"/> -->
-           <!-- <mesh filename="package://ur5_intpro/meshes/visual/robotiq_arg2f_85_base_link_1.dae" /> -->
-           <mesh filename="package://ur5_intpro/meshes/visual/base.dae" />
-        </geometry>
-      </collision>
-    </link>
-  <joint name="robotiq_joint" type="fixed">
-    <parent link="tool0" />
-    <child link = "robotiq_arg2f_base_link" />
-    <origin xyz="0.5 0.0 0.5" rpy="0.0 0.0 0.0" />
- </joint>
-<gazebo reference="robotiq_arg2f_base_link">
-      <mu1 value="1.0"/>
-      <mu2 value="1.0"/>
-      <kp value="900000000.0"></kp>
-      <kd value="800000000.0"></kd>
-  </gazebo>
-<!--  <link name="robotiq_arg2f_base_link">
-    <inertial>
-      <origin xyz="0 0 0" rpy="0 0 0" />
-      <mass value="0.48" />
-      <inertia
-        ixx="6.66"
-        ixy="0"
-        ixz="0"
-        iyy="6.66"
-        iyz="0"
-        izz="6.66" />
-    </inertial>
-     <visual>
+  <xacro:include filename="$(find robotiq_description)/urdf/robotiq_85_gripper.urdf.xacro" />
+  <!-- Robotiq Coupler -->
+  <!--  + Height added by the coupler: 8mm -->
+  <!--  + Reference frame: at the middle (4mm) -->
+  <link name="robotiq_coupler">
+    <visual>
       <geometry>
-        <box size="0.05 0.05 0.05"/>
+        <mesh filename="package://robotiq_description/meshes/robotiq_85_coupler.stl" />
       </geometry>
-      <origin rpy="0 0 0" xyz="0 0 0"/>
+      <material name="flat_black"/>
     </visual>
     <collision>
       <geometry>
-        <box size="0.05 0.05 0.05"/>
+        <mesh filename="package://robotiq_description/meshes/robotiq_85_coupler.stl" />
       </geometry>
-      <origin rpy="0 0 0" xyz="0 0 0"/>
     </collision>
+    <inertial>
+      <origin xyz="2.073e-05   1.45286e-03  -1.1049e-03" rpy="0 0 0" />
+      <mass value="0.168" />
+      <inertia ixx="6.69695624e-05" ixy="5.21511788e-09" ixz="-2.74383009e-08"
+               iyy="7.85088161e-05" iyz="5.41105193e-07" izz="1.41819717e-04"/>
+    </inertial>
   </link>
-   <gazebo reference="robotiq_arg2f_base_link">
-    <mu1 value="1.0"/>
-    <mu2 value="1.0"/>
-    <kp value="900000000.0"></kp>
-    <kd value="800000000.0"></kd>
-    <selfCollide value="false"/>
+  <joint name="robotiq_coupler_joint" type="fixed">
+    <origin xyz="0 0 0.004" rpy="0 0 ${-pi/2.0}" />
+    <parent link="tool0"/>
+    <child link="robotiq_coupler"/>
+  </joint>
+  <gazebo reference="robotiq_coupler">
+    <mu1>0.9</mu1>
+    <mu2>0.9</mu2>
+    <material>Gazebo/FlatBlack</material>
+  </gazebo>
+  <!-- Equivalent to the OpenRAVE manipulator denso_robotiq_85_gripper -->
+  <!-- <link name="denso_robotiq_85_gripper" /> -->
+  <!-- <joint name="manipulator_dummy_joint" type="fixed"> -->
+  <!--   <origin xyz="0 0 0.1441" rpy="0 0 0" /> -->
+  <!--   <parent link="robotiq_coupler"/> -->
+  <!--   <child link="denso_robotiq_85_gripper"/> -->
+  <!-- </joint> -->
+  <!-- Attach the robotiq 85 gripper -->
+  <xacro:robotiq_85_gripper prefix="" parent="robotiq_coupler" >
+    <origin xyz="0 0 0.004" rpy="0 ${-pi/2} ${pi}"/>
+  </xacro:robotiq_85_gripper>
+  <!-- Gazebo FT sensor plugin -->
+  <!-- <gazebo reference="wrist_3_joint">
+    <provideFeedback>true</provideFeedback>
+  </gazebo>
+  <gazebo>
+    <plugin name="ft_sensor_plugin" filename="libgazebo_ros_ft_sensor.so">
+      <updateRate>250.0</updateRate>
+      <topicName>ft_sensor/raw</topicName>
+      <gaussianNoise>0.0</gaussianNoise>
+      <jointName>wrist_3_joint</jointName>
+    </plugin>
+  </gazebo>
+   -->
+  <!-- Gazebo grasping plugin -->
+  <!-- <gazebo>
+    <gripper name="gazebo_gripper">
+      <grasp_check>
+        <attach_steps>2</attach_steps>
+        <detach_steps>2</detach_steps>
+        <min_contact_count>3</min_contact_count>
+      </grasp_check>
+      <gripper_link>robotiq_85_left_finger_tip_link</gripper_link>
+      <gripper_link>robotiq_85_right_finger_tip_link</gripper_link>
+      <palm_link>robotiq_85_base_link</palm_link>
+    </gripper>
   </gazebo> -->
 </robot>
