Commit message: updates and changes for robotiq gripper

File: urdf/custom_ur5.urdf.xacro (robot description, xacro)
@@ -13,6 +13,6 @@
   <xacro:ur5_robot prefix="" joint_limited="true"
     shoulder_pan_lower_limit="${-pi}" shoulder_pan_upper_limit="${pi}"
-    shoulder_lift_lower_limit="${-pi/2.0}" shoulder_lift_upper_limit="${-pi/5.0}"
-    elbow_joint_lower_limit="${pi/5.0}" elbow_joint_upper_limit="${pi}"
+    shoulder_lift_lower_limit="${-pi}" shoulder_lift_upper_limit="${-pi/4}"
+    elbow_joint_lower_limit="${-pi}" elbow_joint_upper_limit="${pi}"
     wrist_1_lower_limit="${-pi}" wrist_1_upper_limit="${pi}"
     wrist_2_lower_limit="${-pi}" wrist_2_upper_limit="${pi}"

File: urdf/kdl_custom_ur5.urdf (robot description, URDF)
Before this commit: robot ur5, 13 links, 12 joints
Links:
- removed link robotiq_arg2f_base_link
- added link robotiq_85_base_link, mass 0.636951; collision mesh filename=package://robotiq_description/meshes/collision/robotiq_85_b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; visual mesh filename=package://robotiq_description/meshes/visual/robotiq_85_base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
- added link robotiq_85_left_finger_link, mass 0.027309; collision mesh filename=package://robotiq_description/meshes/collision/robotiq_85_f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; visual mesh filename=package://robotiq_description/meshes/visual/robotiq_85_fing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
- added link robotiq_85_left_finger_tip_link, mass 0.019555; collision mesh filename=package://robotiq_description/meshes/collision/robotiq_85_f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; visual mesh filename=package://robotiq_description/meshes/visual/robotiq_85_fing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
- added link robotiq_85_left_inner_knuckle_link, mass 0.029951; collision mesh filename=package://robotiq_description/meshes/collision/robotiq_85_i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; visual mesh filename=package://robotiq_description/meshes/visual/robotiq_85_inne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
- added link robotiq_85_left_knuckle_link, mass 0.018491; collision mesh filename=package://robotiq_description/meshes/collision/robotiq_85_k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; visual mesh filename=package://robotiq_description/meshes/visual/robotiq_85_knuc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
- added link robotiq_85_right_finger_link, mass 0.027309; collision mesh filename=package://robotiq_description/meshes/collision/robotiq_85_f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; visual mesh filename=package://robotiq_description/meshes/visual/robotiq_85_fing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
- added link robotiq_85_right_finger_tip_link, mass 0.019555; collision mesh filename=package://robotiq_description/meshes/collision/robotiq_85_f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; visual mesh filename=package://robotiq_description/meshes/visual/robotiq_85_fing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
- added link robotiq_85_right_inner_knuckle_link, mass 0.029951; collision mesh filename=package://robotiq_description/meshes/collision/robotiq_85_i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; visual mesh filename=package://robotiq_description/meshes/visual/robotiq_85_inne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
- added link robotiq_85_right_knuckle_link, mass 0.018491; collision mesh filename=package://robotiq_description/meshes/collision/robotiq_85_k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; visual mesh filename=package://robotiq_description/meshes/visual/robotiq_85_knuc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
- added link robotiq_coupler, mass 0.168; collision mesh filename=package://robotiq_description/meshes/robotiq_85_coupler.stl; visual mesh filename=package://robotiq_description/meshes/robotiq_85_coupler.stl
Joints:
- removed joint robotiq_joint
- added joint robotiq_85_base_joint: type fixed, parent robotiq_coupler, child robotiq_85_base_link, origin xyz=0 0 0.004 rpy=0 -1.57079632679 3.14159265359
- added joint robotiq_85_left_finger_joint: type fixed, parent robotiq_85_left_knuckle_link, child robotiq_85_left_finger_link, origin xyz=-0.00408552455 -0.03148604435 0.0 rpy=0 0 0
- added joint robotiq_85_left_finger_tip_joint: type continuous, parent robotiq_85_left_inner_knuckle_link, child robotiq_85_left_finger_tip_link, origin xyz=0.04303959807 -0.03759940821 0.0 rpy=0.0 0.0 0.0, axis 0 0 1, limit lower=-3.14 upper=3.14 effort=0.1 velocity=100.0, mimic joint=robotiq_85_left_knuckle_joint multiplier=-1
- added joint robotiq_85_left_inner_knuckle_joint: type continuous, parent robotiq_85_base_link, child robotiq_85_left_inner_knuckle_link, origin xyz=0.06142 0.0127 0 rpy=3.14159265359 0.0 0.0, axis 0 0 1, limit lower=-3.14 upper=3.14 effort=0.1 velocity=100.0, mimic joint=robotiq_85_left_knuckle_joint offset=0
- added joint robotiq_85_left_knuckle_joint: type revolute, parent robotiq_85_base_link, child robotiq_85_left_knuckle_link, origin xyz=0.05490451627 0.03060114443 0.0 rpy=3.14159265359 0.0 0.0, axis 0 0 1, limit lower=0.0 upper=0.80285 effort=1000 velocity=0.5
- added joint robotiq_85_right_finger_joint: type fixed, parent robotiq_85_right_knuckle_link, child robotiq_85_right_finger_link, origin xyz=-0.00408552455 -0.03148604435 0.0 rpy=0 0 0
- added joint robotiq_85_right_finger_tip_joint: type continuous, parent robotiq_85_right_inner_knuckle_link, child robotiq_85_right_finger_tip_link, origin xyz=0.04303959807 -0.03759940821  0.0 rpy=0.0 0.0 0.0, axis 0 0 1, limit lower=-3.14 upper=3.14 effort=0.1 velocity=100.0, mimic joint=robotiq_85_left_knuckle_joint multiplier=-1
- added joint robotiq_85_right_inner_knuckle_joint: type continuous, parent robotiq_85_base_link, child robotiq_85_right_inner_knuckle_link, origin xyz=0.06142 -0.0127 0 rpy=0 0 0, axis 0 0 1, limit lower=-3.14 upper=3.14 effort=0.1 velocity=100.0, mimic joint=robotiq_85_left_knuckle_joint offset=0
- added joint robotiq_85_right_knuckle_joint: type continuous, parent robotiq_85_base_link, child robotiq_85_right_knuckle_link, origin xyz=0.05490451627 -0.03060114443 0.0 rpy=0.0 0.0 0.0, axis 0 0 1, limit lower=-3.14 upper=3.14 effort=1000 velocity=100.0, mimic joint=robotiq_85_left_knuckle_joint
- added joint robotiq_coupler_joint: type fixed, parent tool0, child robotiq_coupler, origin xyz=0 0 0.004 rpy=0 0 -1.57079632679
- joint elbow_joint: limit lower=0.628318530718 upper=3.14159265359 effort=150.0 velocity=3.15 -> lower=-3.14159265359 upper=3.14159265359 effort=150.0 velocity=1.57
- joint shoulder_lift_joint: limit lower=-1.57079632679 upper=-0.628318530718 effort=150.0 velocity=3.15 -> lower=-3.14159265359 upper=-0.785398163397 effort=150.0 velocity=1.57
- joint shoulder_pan_joint: limit lower=-3.14159265359 upper=3.14159265359 effort=150.0 velocity=3.15 -> lower=-3.14159265359 upper=3.14159265359 effort=150.0 velocity=1.57; origin xyz=0.0 0.0 0.089159 rpy=0.0 0.0 0.0 -> xyz=0.0 0.0 0.089159 rpy=0.0 0.0 -0.785398163397

File: urdf/ur5.urdf.xacro (robot description, xacro)
@@ -13,7 +13,7 @@
   </xacro:macro>
   <xacro:macro name="ur5_robot" params="prefix joint_limited
-    shoulder_pan_lower_limit:=${-pi}    shoulder_pan_upper_limit:=${pi}
-    shoulder_lift_lower_limit:=${-pi}    shoulder_lift_upper_limit:=${pi}
-    elbow_joint_lower_limit:=${-pi}    elbow_joint_upper_limit:=${pi}
+    shoulder_pan_lower_limit:=${-pi/3}    shoulder_pan_upper_limit:=${pi/3}
+    shoulder_lift_lower_limit:=${-pi/2.0}    shoulder_lift_upper_limit:=${-pi/2.0 + 0.01}
+    elbow_joint_lower_limit:=${-pi/3.0}    elbow_joint_upper_limit:=${0}
     wrist_1_lower_limit:=${-pi}    wrist_1_upper_limit:=${pi}
     wrist_2_lower_limit:=${-pi}    wrist_2_upper_limit:=${pi}
@@ -102,11 +102,11 @@
       <axis xyz="0 0 1" />
       <xacro:unless value="${joint_limited}">
-        <limit lower="${-2.0 * pi}" upper="${2.0 * pi}" effort="150.0" velocity="3.15"/>
-        <xacro:if value="${safety_limits}">
-          <safety_controller soft_lower_limit="${-2.0 * pi + safety_pos_margin}" soft_upper_limit="${2.0 * pi - safety_pos_margin}" k_position="${safety_k_position}" k_velocity="0.0"/>
-        </xacro:if>
-      </xacro:unless>
-      <xacro:if value="${joint_limited}">
-        <limit lower="${shoulder_pan_lower_limit}" upper="${shoulder_pan_upper_limit}" effort="150.0" velocity="3.15"/>
+        <limit lower="${-2.0 * pi}" upper="${2.0 * pi}" effort="150.0" velocity="1.57"/>
+        <xacro:if value="${safety_limits}">
+          <safety_controller soft_lower_limit="${-2.0 * pi + safety_pos_margin}" soft_upper_limit="${2.0 * pi - safety_pos_margin}" k_position="${safety_k_position}" k_velocity="0.0"/>
+        </xacro:if>
+      </xacro:unless>
+      <xacro:if value="${joint_limited}">
+        <limit lower="${shoulder_pan_lower_limit}" upper="${shoulder_pan_upper_limit}" effort="150.0" velocity="1.57"/>
         <xacro:if value="${safety_limits}">
           <safety_controller soft_lower_limit="${shoulder_pan_lower_limit + safety_pos_margin}" soft_upper_limit="${shoulder_pan_upper_limit - safety_pos_margin}" k_position="${safety_k_position}" k_velocity="0.0"/>
@@ -139,11 +139,11 @@
       <axis xyz="0 1 0" />
       <xacro:unless value="${joint_limited}">
-        <limit lower="${-2.0 * pi}" upper="${2.0 * pi}" effort="150.0" velocity="3.15"/>
-        <xacro:if value="${safety_limits}">
-          <safety_controller soft_lower_limit="${-2.0 * pi + safety_pos_margin}" soft_upper_limit="${2.0 * pi - safety_pos_margin}" k_position="${safety_k_position}" k_velocity="0.0"/>
-        </xacro:if>
-      </xacro:unless>
-      <xacro:if value="${joint_limited}">
-        <limit lower="${shoulder_lift_lower_limit}" upper="${shoulder_lift_upper_limit}" effort="150.0" velocity="3.15"/>
+        <limit lower="${-2.0 * pi}" upper="${2.0 * pi}" effort="150.0" velocity="1.57"/>
+        <xacro:if value="${safety_limits}">
+          <safety_controller soft_lower_limit="${-2.0 * pi + safety_pos_margin}" soft_upper_limit="${2.0 * pi - safety_pos_margin}" k_position="${safety_k_position}" k_velocity="0.0"/>
+        </xacro:if>
+      </xacro:unless>
+      <xacro:if value="${joint_limited}">
+        <limit lower="${shoulder_lift_lower_limit}" upper="${shoulder_lift_upper_limit}" effort="150.0" velocity="1.57"/>
         <xacro:if value="${safety_limits}">
           <safety_controller soft_lower_limit="${shoulder_lift_lower_limit + safety_pos_margin}" soft_upper_limit="${shoulder_lift_upper_limit - safety_pos_margin}" k_position="${safety_k_position}" k_velocity="0.0"/>
@@ -176,11 +176,11 @@
       <axis xyz="0 1 0" />
       <xacro:unless value="${joint_limited}">
-        <limit lower="${-pi}" upper="${pi}" effort="150.0" velocity="3.15"/>
-        <xacro:if value="${safety_limits}">
-          <safety_controller soft_lower_limit="${-2.0 * pi + safety_pos_margin}" soft_upper_limit="${2.0 * pi - safety_pos_margin}" k_position="${safety_k_position}" k_velocity="0.0"/>
-        </xacro:if>
-      </xacro:unless>
-      <xacro:if value="${joint_limited}">
-        <limit lower="${elbow_joint_lower_limit}" upper="${elbow_joint_upper_limit}" effort="150.0" velocity="3.15"/>
+        <limit lower="${-pi}" upper="${pi}" effort="150.0" velocity="1.57"/>
+        <xacro:if value="${safety_limits}">
+          <safety_controller soft_lower_limit="${-2.0 * pi + safety_pos_margin}" soft_upper_limit="${2.0 * pi - safety_pos_margin}" k_position="${safety_k_position}" k_velocity="0.0"/>
+        </xacro:if>
+      </xacro:unless>
+      <xacro:if value="${joint_limited}">
+        <limit lower="${elbow_joint_lower_limit}" upper="${elbow_joint_upper_limit}" effort="150.0" velocity="1.57"/>
         <xacro:if value="${safety_limits}">
           <safety_controller soft_lower_limit="${elbow_joint_lower_limit + safety_pos_margin}" soft_upper_limit="${elbow_joint_upper_limit - safety_pos_margin}" k_position="${safety_k_position}" k_velocity="0.0"/>

Commit message: working shadow and sim gripper action

File: urdf/custom_ur5.urdf.xacro (robot description, xacro)
@@ -41,11 +41,11 @@
         izz="6666.66" />
     </inertial>
-     <visual>
-      <geometry>
+     <!-- <visual> -->
+      <!-- <geometry> -->
         <!-- <box size="2.0 2.0 1.0"/> -->
-        <mesh filename="package://ur5_intpro/meshes/table/table.dae" />
-      </geometry>
-      <origin rpy="0 0 0" xyz="0 0 0"/>
-    </visual>
+        <!-- <mesh filename="package://ur5_intpro/meshes/table/table.dae" /> -->
+      <!-- </geometry> -->
+      <!-- <origin rpy="0 0 0" xyz="0 0 0"/> -->
+    <!-- </visual> -->
     <collision>
       <geometry>

Commit message: working for 203-03 lab

File: urdf/custom_ur5.urdf.xacro (robot description, xacro)
@@ -13,9 +13,9 @@
   <xacro:ur5_robot prefix="" joint_limited="true"
     shoulder_pan_lower_limit="${-pi}" shoulder_pan_upper_limit="${pi}"
-    shoulder_lift_lower_limit="${-pi}" shoulder_lift_upper_limit="${-pi/4}"
+    shoulder_lift_lower_limit="${-pi}" shoulder_lift_upper_limit="${-pi/8}"
     elbow_joint_lower_limit="${-pi}" elbow_joint_upper_limit="${pi}"
     wrist_1_lower_limit="${-pi}" wrist_1_upper_limit="${pi}"
     wrist_2_lower_limit="${-pi}" wrist_2_upper_limit="${pi}"
-    wrist_3_lower_limit="${-pi}" wrist_3_upper_limit="${pi}"
+    wrist_3_lower_limit="${-2*pi}" wrist_3_upper_limit="${2*pi}"
     transmission_hw_interface="$(arg transmission_hw_interface)"
   />
@@ -138,3 +138,26 @@
     </gripper>
   </gazebo> -->
+<!-- fake end effector -->
+<link name="fake_end_effector_link">
+    <visual>
+    <geometry>
+      <box size="0.01 0.01 0.01"/>
+    </geometry>
+    <origin rpy="0 0 0" xyz="0 0 0"/>
+    <material name="red"/>
+  </visual>
+    <collision>
+    <geometry>
+      <box size="0 0 0"/>
+    </geometry>
+    <origin rpy="0 0 0" xyz="0 0 0"/>
+  </collision>
+  </link>
+  <joint name="fake_end_effector_joint" type="fixed">
+    <origin rpy="0 0 0" xyz="0.145 0 0"/>
+    <!-- <origin rpy="0 0 0" xyz="0 0.1 0"/> -->
+    <!-- <parent link="J6"/> -->
+    <parent link="robotiq_85_base_link"/>
+    <child link="fake_end_effector_link"/>
+  </joint>
 </robot>

File: urdf/ur5.urdf.xacro (robot description, xacro)
@@ -98,6 +98,6 @@
       <parent link="${prefix}base_link" />
       <child link = "${prefix}shoulder_link" />
-      <!-- <origin xyz="0.0 0.0 ${shoulder_height}" rpy="0.0 0.0 0.0" /> -->
-      <origin xyz="0.0 0.0 ${shoulder_height}" rpy="0.0 0.0 ${-pi/4.0}" />
+      <origin xyz="0.0 0.0 ${shoulder_height}" rpy="0.0 0.0 0.0" />
+      <!-- <origin xyz="0.0 0.0 ${shoulder_height}" rpy="0.0 0.0 ${-pi/4.0}" /> -->
       <axis xyz="0 0 1" />
       <xacro:unless value="${joint_limited}">

Commit message: now listen to generated goal from intention projection

File: urdf/custom_ur5.urdf.xacro (robot description, xacro)
@@ -142,5 +142,8 @@
     <visual>
     <geometry>
-      <box size="0.01 0.01 0.01"/>
+      <box size="0.06 0.06 0.06"/>
+      <!-- <mesh filename="package://ur5_intpro/meshes/visualize.stl" /> -->
+      <!-- <mesh filename="package://ur5_intpro/meshes/visualize.dae" /> -->
+      <!-- <box size="0.01 0.01 0.01"/> -->
     </geometry>
     <origin rpy="0 0 0" xyz="0 0 0"/>
@@ -155,5 +158,5 @@
   </link>
   <joint name="fake_end_effector_joint" type="fixed">
-    <origin rpy="0 0 0" xyz="0.145 0 0"/>
+    <origin rpy="0 0 0" xyz="0.145 0.0 0.0"/>
     <!-- <origin rpy="0 0 0" xyz="0 0.1 0"/> -->
     <!-- <parent link="J6"/> -->
@@ -161,3 +164,11 @@
     <child link="fake_end_effector_link"/>
   </joint>
+<material name="orange">
+    <color rgba="${255/255} ${108/255} ${10/255} 1.0"/>
+</material>
+    <gazebo reference="fake_end_effector_link">
+    <mu1>0.9</mu1>
+    <mu2>0.9</mu2>
+    <material>Gazebo/Orange</material>
+  </gazebo>
 </robot>
