Commit message: updated scripts

File: urdf/custom_ur5.urdf (robot description, URDF)
Before this commit: robot ur5, 23 links, 22 joints
Links:
- link robotiq_85_base_link: mass 0.636951 -> None
- link robotiq_85_left_finger_link: mass 0.027309 -> None
- link robotiq_85_left_finger_tip_link: mass 0.019555 -> None
- link robotiq_85_left_inner_knuckle_link: mass 0.029951 -> None
- link robotiq_85_left_knuckle_link: mass 0.018491 -> None
- link robotiq_85_right_finger_link: mass 0.027309 -> None
- link robotiq_85_right_finger_tip_link: mass 0.019555 -> None
- link robotiq_85_right_inner_knuckle_link: mass 0.029951 -> None
- link robotiq_85_right_knuckle_link: mass 0.018491 -> None
- link robotiq_coupler: mass 0.168 -> None
